File: hardware/main-board/ecoconnect-main-board.kicad_pcb (KiCad board)
At the start: 4 copper layers, 56 x 72 mm, 26 parts, among them J1 BATT Conn, J2 Conn_01x08_Socket, J3 Conn_Coaxial, J4 Conn_01x08_Socket, J5 Conn_01x12_MountingPin, J6 Conn_01x12_Socket, J7 Conn_02x03_Top_Bottom, J8 Conn_01x08_Socket, M2 A660-900T22, Q1 AO3401A, Q2 AO3401A, SW1 SW_Omron_B3FS, SW2 SW_Reed

Commit message: Add Japanese-first docs with English locale switcher.
Keep EcoCONNECT, hollyRock, Raspberry Pi Pico, and STEAM as English product names in JA copy.

Co-authored-by: Cursor <cursoragent@cursor.com>
Parts:
- CR1: footprint hollyRock:D5V0F1U2S9 -> auralinc:D5V0F1U2S9
- F1: footprint MINISMDC075F-2 resettable Fuse:FUS_MINISMDC075F_TYCO_TYC -> auralinc:FUS_MINISMDC075F_TYCO_TYC
- U1: footprint MCU_RaspberryPi_and_Boards:RPi_Pico_SMD_TH -> auralinc:RPi_Pico_SMD_TH
Other:
- board text removed: "Have fun!"
