File: hardware/main-board/ecoconnect-main-board.kicad_sch (KiCad schematic)
At the start: 26 parts, among them J1 BATT Conn, J2 Conn_01x08_Socket, J3 Conn_Coaxial, J4 Conn_01x08_Socket, J5 Conn_01x12_MountingPin, J6 Conn_01x12_Socket, J7 Conn_02x03_Top_Bottom, J8 Conn_01x08_Socket, M2 A660-900T22, Q1 AO3401A, Q2 AO3401A, SW1 SW_Omron_B3FS, SW2 SW_Reed

Commit message: Add Japanese-first docs with English locale switcher.
Keep EcoCONNECT, hollyRock, Raspberry Pi Pico, and STEAM as English product names in JA copy.

Co-authored-by: Cursor <cursoragent@cursor.com>
Parts:
- CR1: footprint hollyRock:D5V0F1U2S9 -> auralinc:D5V0F1U2S9; symbol D5V0F1U2S9:D5V0F1U2S9-7 -> auralinc:D5V0F1U2S9-7
- F1: footprint MINISMDC075F-2 resettable Fuse:FUS_MINISMDC075F_TYCO_TYC -> auralinc:FUS_MINISMDC075F_TYCO_TYC
- M1: symbol hollyrock_lib:A660-900T22-EV1 -> auralinc:A660-900T22-EV1
- M2: symbol hollyrock_lib:A660-900T22 -> auralinc:A660-900T22
- U1: footprint MCU_RaspberryPi_and_Boards:RPi_Pico_SMD_TH -> auralinc:RPi_Pico_SMD_TH; symbol hollyRockDBLib:LSI/MCU_RASP_Pico2_wo_WB -> auralinc:Pico
Changed lines of the file:
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@@
 		(title "AuraLinc Project")
 		(date "2026-08-29")
-		(rev "0.4.1")
+		(rev "0.5.0")
 		(company "hollyRock")
 	)
@@
 	)
 	(symbol
-		(lib_id "hollyrock_lib:A660-900T22-EV1")
+		(lib_id "auralinc:A660-900T22-EV1")
 		(at 90.17 96.52 0)
 		(unit 1)
@@
 	)
 	(symbol
-		(lib_id "hollyrock_lib:A660-900T22")
+		(lib_id "auralinc:A660-900T22")
 		(at 95.25 58.42 0)
 		(unit 1)
@@
 	)
 	(symbol
-		(lib_id "hollyRockDBLib:LSI/MCU_RASP_Pico2_wo_WB")
+		(lib_id "auralinc:Pico")
 		(at 195.58 72.39 270)
 		(unit 1)
@@
 			)
 		)
-		(property "Footprint" "MCU_RaspberryPi_and_Boards:RPi_Pico_SMD_TH"
+		(property "Footprint" "auralinc:RPi_Pico_SMD_TH"
 			(at 195.58 72.39 90)
 			(effects
@@
 		(property "Datasheet" ""
 			(at 195.58 72.39 0)
-			(show_name yes)
 			(effects
 				(font
@@
 	)
 	(symbol
-		(lib_id "D5V0F1U2S9:D5V0F1U2S9-7")
+		(lib_id "auralinc:D5V0F1U2S9-7")
 		(at 34.29 168.91 0)
 		(unit 1)
@@
 			)
 		)
-		(property "Footprint" "hollyRock:D5V0F1U2S9"
+		(property "Footprint" "auralinc:D5V0F1U2S9"
 			(at 34.29 168.91 0)
 			(effects
@@
 			)
 		)
-		(property "Footprint" "MINISMDC075F-2  resettable Fuse:FUS_MINISMDC075F_TYCO_TYC"
+		(property "Footprint" "auralinc:FUS_MINISMDC075F_TYCO_TYC"
 			(at 53.34 156.21 0)
 			(effects
